Commit message: ready to fix openarm right arm's left finger none collision problem

File: source/isaaclab_assets/data/v1_camera_isaac/urdf/v1_camera_original.urdf (robot description, URDF)
Before this commit: robot openarm, 26 links, 25 joints
Links:
- link openarm_left_link0: geometry collision mesh filename=package://v1_camera_isaac/mesh/arm/collision/link0_symp.stl scale=0.001 -0.001 0.001; visual mesh filename=package://v1_camera_isaac/mesh/arm/visual/link0.dae scale=0.001 -0.001 0.001
- link openarm_left_link1: geometry collision mesh filename=package://v1_camera_isaac/mesh/arm/collision/link1_symp.stl scale=0.001 -0.001 0.001; visual mesh filename=package://v1_camera_isaac/mesh/arm/visual/link1.dae scale=0.001 -0.001 0.001
- link openarm_left_link2: geometry collision mesh filename=package://v1_camera_isaac/mesh/arm/collision/link2_symp.stl scale=0.001 -0.001 0.001; visual mesh filename=package://v1_camera_isaac/mesh/arm/visual/link2.dae scale=0.001 -0.001 0.001
- link openarm_left_link5: geometry collision mesh filename=package://v1_camera_isaac/mesh/arm/collision/link5_symp.stl scale=0.001 -0.001 0.001; visual mesh filename=package://v1_camera_isaac/mesh/arm/visual/link5.dae scale=0.001 -0.001 0.001
- link openarm_left_link6: geometry collision mesh filename=package://v1_camera_isaac/mesh/arm/collision/link6_symp.stl scale=0.001 -0.001 0.001; visual mesh filename=package://v1_camera_isaac/mesh/arm/visual/link6.dae scale=0.001 -0.001 0.001
- link openarm_left_link7: geometry collision mesh filename=package://v1_camera_isaac/mesh/arm/collision/link7_symp.stl scale=0.001 -0.001 0.001; visual mesh filename=package://v1_camera_isaac/mesh/arm/visual/link7.dae scale=0.001 -0.001 0.001
- link openarm_left_right_finger: geometry collision mesh filename=package://v1_camera_isaac/mesh/end_effector/parallel_link/m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 scale=0.001 -0.001 0.001; visual mesh filename=package://v1_camera_isaac/mesh/end_effector/parallel_link/m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 scale=0.001 -0.001 0.001
- link openarm_right_right_finger: geometry collision mesh filename=package://v1_camera_isaac/mesh/end_effector/parallel_link/m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 scale=0.001 -0.001 0.001; visual mesh filename=package://v1_camera_isaac/mesh/end_effector/parallel_link/m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 scale=0.001 -0.001 0.001

File: source/isaaclab_assets/data/v1_camera_isaac/urdf/v1_camera_test.urdf (robot description, URDF)
Before this commit: robot openarm, 26 links, 25 joints
Links:
- link openarm_left_link0: geometry collision mesh filename=package://v1_camera_isaac/mesh/arm/collision/link0_symp.stl scale=0.001 -0.001 0.001; visual mesh filename=package://v1_camera_isaac/mesh/arm/visual/link0.dae scale=0.001 -0.001 0.001
- link openarm_left_link1: geometry collision mesh filename=package://v1_camera_isaac/mesh/arm/collision/link1_symp.stl scale=0.001 -0.001 0.001; visual mesh filename=package://v1_camera_isaac/mesh/arm/visual/link1.dae scale=0.001 -0.001 0.001
- link openarm_left_link2: geometry collision mesh filename=package://v1_camera_isaac/mesh/arm/collision/link2_symp.stl scale=0.001 -0.001 0.001; visual mesh filename=package://v1_camera_isaac/mesh/arm/visual/link2.dae scale=0.001 -0.001 0.001
- link openarm_left_link5: geometry collision mesh filename=package://v1_camera_isaac/mesh/arm/collision/link5_symp.stl scale=0.001 -0.001 0.001; visual mesh filename=package://v1_camera_isaac/mesh/arm/visual/link5.dae scale=0.001 -0.001 0.001
- link openarm_left_link6: geometry collision mesh filename=package://v1_camera_isaac/mesh/arm/collision/link6_symp.stl scale=0.001 -0.001 0.001; visual mesh filename=package://v1_camera_isaac/mesh/arm/visual/link6.dae scale=0.001 -0.001 0.001
- link openarm_left_link7: geometry collision mesh filename=package://v1_camera_isaac/mesh/arm/collision/link7_symp.stl scale=0.001 -0.001 0.001; visual mesh filename=package://v1_camera_isaac/mesh/arm/visual/link7.dae scale=0.001 -0.001 0.001
- link openarm_left_right_finger: geometry collision mesh filename=package://v1_camera_isaac/mesh/end_effector/parallel_link/m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 scale=0.001 -0.001 0.001; visual mesh filename=package://v1_camera_isaac/mesh/end_effector/parallel_link/m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 scale=0.001 -0.001 0.001
- link openarm_right_right_finger: geometry collision mesh filename=package://v1_camera_isaac/mesh/end_effector/parallel_link/m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 scale=0.001 -0.001 0.001; visual mesh filename=package://v1_camera_isaac/mesh/end_effector/parallel_link/m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 scale=0.001 -0.001 0.001
