Commit message: dataset generation on going...

File: source/isaaclab_assets/data/v1_camera_isaac/urdf/v1_camera.urdf (robot description, URDF)
Before this commit: robot openarm, 26 links, 25 joints
Links:
- link openarm_left_camera_link: geometry collision box size=0.0101 0.0238 0.0336; collision box size=0.0288 0.0912 0.0336
- link openarm_right_camera_link: geometry collision box size=0.0101 0.0238 0.0336; collision box size=0.0288 0.0912 0.0336
