Commit message: Claude generated: real-rig OpenArm in sim (gripper, camera mount, look, Mimic-v1, DR on the look)
Robot model (scripts/tools/sysid, applied as USD sublayers; the robot's USDs are gitignored):
- add_openarm_hand.py: the official parallel-gripper hand (rail housing) on link7, official finger
  joint offsets (+-5 mm), 4.3 mm foam pads on the fingertips (measured: real pads open to ~77.8 mm),
  joint lower limit where the pads meet (no clipping when closed on nothing); URDF to match.
- add_openarm_camera_mount.py: real D435i bar + clamp ring halves (d435i_*.stl), housing off-centre
  and turned to the sensor's view axis, USB plug and cable, aluminium/black-glass housing materials.
- Wrist cameras: lens on the housing face, near clip 1 mm, far clip 4 m (room walls); Fabric
  camera-mount sync event (mdp/openarm_camera_mount.py).

Scene and task:
- Black workspace mats from the real rig (openarm_workspace_mat.py); recording spawn closer to the body
  with hand keep-out boxes; robot self-collisions off by default (OPENARM_SELF_COLLISIONS=1 to enable).
- Can size kept at 0.8; size-derived constants; grip thresholds re-measured for the padded gripper.

Real look (data/real2sim/pringles_v00):
- Room backdrop fused from ~2600 real frames of all three cameras (build_room_backdrop.py), body
  backdrop trimmed to the table, robot colours refit; old wrist posters in superseded/.
- Contact physics as a startup event, camera blur/noise inside the observations.
- Isaac-PickUp-RedCube-OpenArm-IK-Abs-Mimic-v1; domain randomization on the look
  (openarm_real_look_randomization.py): light relative to the look and carried onto the backdrop,
  skybox swap hides the room, table tint; pad height moves the photo table; wrist-camera jitter
  never moves the lens into the housing.

Co-Authored-By: Claude Opus 5.5 <noreply@anthropic.com>

File: source/isaaclab_assets/data/v1_camera_isaac/urdf/v1_camera.urdf (robot description, URDF)
Before this commit: robot openarm, 26 links, 25 joints
Joints:
- joint openarm_left_finger_joint1: limit lower=0.0 upper=0.044 effort=333 velocity=10.0 -> lower=0.00506 upper=0.044 effort=333 velocity=10.0; origin xyz=0.0 0.0 0.1025 rpy=0 0 0 -> xyz=0.0 -0.005 0.1025 rpy=0 0 0
- joint openarm_left_finger_joint2: limit lower=0.0 upper=0.044 effort=333 velocity=10.0 -> lower=0.00506 upper=0.044 effort=333 velocity=10.0; origin xyz=0.0 -0.0 0.1025 rpy=0 0 0 -> xyz=0.0 0.005 0.1025 rpy=0 0 0
- joint openarm_right_finger_joint1: limit lower=0.0 upper=0.044 effort=333 velocity=10.0 -> lower=0.00506 upper=0.044 effort=333 velocity=10.0; origin xyz=0.0 0.0 0.1025 rpy=0 0 0 -> xyz=0.0 -0.005 0.1025 rpy=0 0 0
- joint openarm_right_finger_joint2: limit lower=0.0 upper=0.044 effort=333 velocity=10.0 -> lower=0.00506 upper=0.044 effort=333 velocity=10.0; origin xyz=0.0 -0.0 0.1025 rpy=0 0 0 -> xyz=0.0 0.005 0.1025 rpy=0 0 0
